File: BF-AVR/BF-AVR.kicad_sch (KiCad schematic)
At the start: 24 parts, among them J1 USB_B, J10 Conn_01x01_Socket, J11 Conn_01x01_Socket, J12 DE15_Socket_HighDensity_Mount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, J13 Conn_01x01_Socket, J14 Conn_01x01_Socket, J15 Mini-DIN-6, J16 Conn_01x15_Socket, J17 Conn_01x06_Socket, J2 Conn_01x01_Socket, J3 Conn_01x01_Socket, J4 Conn_01x03_Pin, J5 Conn_02x14_Counter_Clockwise, J6 Conn_01x03_Pin, J7 Conn_01x03_Pin, J8 Conn_01x14_Socket, J9 Conn_01x14_Socket, SW1 SW_RESET

Commit message: a
Parts:
- removed J10, J11, J13, J14: Conn_01x01_Socket, Connector_PinHeader_1.00mm:PinHeader_1x01_P1.00mm_Vertical, symbol Connector:Conn_01x01_Socket
- added J10, J11: Conn_01x02_Socket, Connector_PinSocket_2.54mm:PinSocket_1x02_P2.54mm_Vertical, symbol Connector:Conn_01x02_Socket
- J13: renamed from J15; footprint (none) -> Connector_Mini-DIN:Connector_Mini-DIN_Female_6Pin_2rows
- J14: renamed from J16; footprint (none) -> Connector_PinSocket_2.54mm:PinSocket_1x15_P2.54mm_Vertical
- J15: renamed from J17; footprint (none) -> Connector_PinSocket_2.54mm:PinSocket_1x06_P2.54mm_Vertical
- J2, J3: footprint Connector_PinHeader_1.00mm:PinHeader_1x01_P1.00mm_Vertical -> Connector_PinSocket_2.54mm:PinSocket_1x01_P2.54mm_Vertical
- J4, J6, J7: footprint (none) -> Connector_PinHeader_2.54mm:PinHeader_1x03_P2.54mm_Vertical
- J5: footprint (none) -> Package_DIP:DIP-28_W7.62mm
- J8, J9: footprint (none) -> Connector_PinSocket_2.54mm:PinSocket_1x14_P2.54mm_Vertical
Connections:
- net D+: now also J10.1 (Pin_1)
- net D-: now also J10.2 (Pin_2)
- net GND: now also J11.2 (Pin_2)
- net PF6: now also J9.11 (Pin_11)
- net RESET: no longer J9.11 (Pin_11)
- net VCC: now also J11.1 (Pin_1)
